File: Arduino_KNX_Shield.kicad_pcb (KiCad board)
At the start: 2 copper layers, 68.5 x 53.4 mm, 10 parts, among them J1 Conn_01x08_Male, J10 Conn_01x06_Male, J2 Conn_01x10_Male, J3 Conn_01x06_Male, J4 Conn_01x08_Male, J5 KNX, J6 Conn_01x06_Male, J7 Conn_01x06_Male, J8 Conn_01x06_Male, J9 Conn_01x03_Male

Commit message: V.2.2
Other:
- board text added: "© 2021 André Husken | V.2.2 www.arduino-smarthome.de"
- board text removed: "© 2021 André Husken | V.2.1 www.arduino-smarthome.de"
Changed lines of the file:
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@@
     (effects (font (size 0.7 0.7) (thickness 0.1)) (justify right))
   )
-  (gr_text "© 2021 André Husken | V.2.1\nwww.arduino-smarthome.de" (at 141.3891 93.4212 270) (layer F.SilkS)
+  (gr_text "© 2021 André Husken | V.2.2\nwww.arduino-smarthome.de" (at 141.3891 93.4212 270) (layer F.SilkS)
     (effects (font (size 0.7 0.7) (thickness 0.1)))
   )
